Commit message: Correções na descrição

File: pioneer3dx_description/urdf/gazebo_configs.xacro (robot description, xacro)
@@ -65,6 +65,6 @@
         <plugin name="diff_drive" filename="libgazebo_ros_diff_drive.so">
             <!-- Wheel Information -->
-            <left_joint>left_wheel_joint</left_joint>
-            <right_joint>right_wheel_joint</right_joint>
+            <left_joint>base_left_wheel_joint</left_joint>
+            <right_joint>base_right_wheel_joint</right_joint>
             <wheel_separation>0.39</wheel_separation>
             <wheel_diameter>0.15</wheel_diameter>

File: pioneer3dx_description/urdf/robot_core.xacro (robot description, xacro)
@@ -155,5 +155,5 @@
 		</collision>
 	</link>
-	<joint name="swivel_hubcap_joint" type="continuous">
+	<joint name="swivel_hubcap_joint" type="fixed">
 		<origin xyz="-0.026 0 -0.016" rpy="0 0 0" />
 		<axis xyz="0 1 0" />
